Commit message: test(collision): DTC scene Phase B — work-object env, EE bake, SRDF ACM, FCL==OptiX
- Bake the ee_hilok end-effector as a collision mesh on the tool-changer tip
  link (the DTC app attaches it at runtime), so it flows through both backends
  as robot geometry.
- tests/support/dtc_scene.hpp: shared builder used by the DTC test (and, next,
  the benchmark + visualizer) — robot loader, work-object environment
  (mesh.stl + 3 fiducial markers at the app's world poses), an SRDF
  disable_collisions -> AllowedCollisionMatrix parser, and a random-pose sampler.
- test_dtc_scene: SRDF ACM loads (22 pairs); the work-object env builds with a
  genuine collision mix (4.1% of 1000 random 7-DOF poses); and FCL vs OptiX
  agree config-for-config on robot-vs-environment (0 disagreements, mix of
  collide/free). The OptiX case skips cleanly when the backend is not built.

dev-cpu 3/3 (+1 skip); dev-optix DtcScene 4/4 via ctest.

Co-Authored-By: Claude Opus 4.8 <noreply@anthropic.com>

File: tests/fixtures/robots/rbrobout.urdf (robot description, URDF)
Before this commit: robot rbrobout, 17 links, 16 joints
Links:
- link tool_changer_robot_link: geometry collision cylinder length=0.01895 radius=0.0315; collision mesh filename=package://dtc_test/meshes/ee_hilok_collision.stl
