Commit message: fix(fixtures): rbrobout_inlet — jointA TCP frame link + silence dresskit_2 visual error
Adds ee_9636_jA_tcp, a massless frame link fixed to tool_changer_robot_link
at the DTC app's mesh_pose * tcp_pose composition (xyz -0.0154998 0.285
0.2116998; the two 180deg-about-Y rotations cancel to identity within 6e-7
rad) so IK/planning can target the attached jointA EE tip directly instead
of hand-composing the offset (as inlet_ik_visualize.cpp does). No collision
geometry -> scene and SRDF behavior unchanged. Also removes dresskit_2's
empty <visual><geometry> (its mesh line was commented out; urdfdom printed
'Geometry tag contains no child element' on every load).

Verified: full ctest suite green; studio smoke test IK-solves to an FK
target on the new frame.

Co-Authored-By: Claude Fable 5 <noreply@anthropic.com>

File: tests/fixtures/robots/rbrobout_inlet.urdf (robot description, URDF)
Before this commit: robot bmt_9636, 31 links, 30 joints
Links:
- added link ee_9636_jA_tcp
Joints:
- added joint ee_9636_jA_tcp_joint: type fixed, parent tool_changer_robot_link, child ee_9636_jA_tcp, origin xyz=-0.0154998 0.285 0.2116998 rpy=0 0 0
